Commit message: Final hand-in commit

File: src/franka_description/robots/panda_arm.xacro (robot description, xacro)
@@ -10,7 +10,8 @@
   <xacro:property name="mass_link6" value="1.46736" />
   <xacro:property name="mass_link7" value="0.45606" />
-  <xacro:property name="mass_link8" value="0.001" />
-  <!-- Wrong masses to test adaptability of the algorithms, on purpose off by 20% -->
-  <!--xacro:property name="mass_link0" value="3.66357" />
+  <xacro:property name="mass_link8" value="0.1" />
+  <!--xacro:property name="mass_link8" value="0.001" /-->
+  <!-- Wrong masses to test adaptability of the algorithms, on purpose off by 20%
+  <xacro:property name="mass_link0" value="3.66357" />
   <xacro:property name="mass_link1" value="2.04471" />
   <xacro:property name="mass_link2" value="2.56414" />
@@ -20,5 +21,15 @@
   <xacro:property name="mass_link6" value="1.66736" />
   <xacro:property name="mass_link7" value="0.75606" />
-  <xacro:property name="mass_link8" value="0.1" /-->
+  <xacro:property name="mass_link8" value="0.1" /> -->
+  <!-- Wrong masses to test adaptability of the algorithms, on purpose off by 20% mine
+  <xacro:property name="mass_link0" value="3.676284" />
+  <xacro:property name="mass_link1" value="2.813652" />
+  <xacro:property name="mass_link2" value="2.836968" />
+  <xacro:property name="mass_link3" value="2.8566" />
+  <xacro:property name="mass_link4" value="2.913048" />
+  <xacro:property name="mass_link5" value="4.195332" />
+  <xacro:property name="mass_link6" value="1.760832" />
+  <xacro:property name="mass_link7" value="0.547272" />
+  <xacro:property name="mass_link8" value="0.1" />  -->
   <xacro:property name="link0_cog" value="-0.029190 -0.000879 0.056603" />
   <xacro:property name="link1_cog" value="0.000011 -0.031266 -0.069373" />
